File: Connectors1.sch (KiCad schematic (older format))
At the start: 4 parts

Commit message: wiring done ... no DRC errors
Parts:
- removed J?: Conn_01x09_MountingPin, symbol Connector_Generic_MountingPin:Conn_01x09_MountingPin
- removed J? (x2): Conn_01x04_MountingPin, symbol Connector_Generic_MountingPin:Conn_01x04_MountingPin
- removed J?: Conn_02x03_Odd_Even, symbol Connector_Generic:Conn_02x03_Odd_Even
- added J1: Serial, Connector_PinHeader_2.54mm:PinHeader_1x04_P2.54mm_Vertical, symbol Connector_Generic:Conn_01x04
- added J2: Digital pins, Connector_PinHeader_2.54mm:PinHeader_1x09_P2.54mm_Vertical, symbol Connector_Generic:Conn_01x09
- added J3: ICSP, Connector_PinHeader_2.54mm:PinHeader_2x03_P2.54mm_Vertical, symbol Connector_Generic:Conn_02x03_Odd_Even
- added J4: I2C, Connector_PinHeader_2.54mm:PinHeader_1x04_P2.54mm_Vertical, symbol Connector_Generic:Conn_01x04
Connections:
- new net D2: J2.1 (Pin_1)
- new net D3: J2.2 (Pin_2)
- new net D4: J2.3 (Pin_3)
- new net D5: J2.4 (Pin_4)
- new net D6: J2.5 (Pin_5)
- new net D7: J2.6 (Pin_6)
- new net D8: J2.7 (Pin_7)
- new net GND: J1.1 (Pin_1), J2.8 (Pin_8), J3.6 (Pin_6), J4.1 (Pin_1)
- new net MISO: J3.1 (Pin_1)
- new net MOSI: J3.4 (Pin_4)
- new net RST: J3.5 (Pin_5)
- new net RX: J1.3 (Pin_3)
- new net SCK: J3.3 (Pin_3), J4.4 (Pin_4)
- new net SDA: J4.3 (Pin_3)
- new net TX: J1.4 (Pin_4)
- new net VCC: J1.2 (Pin_2), J2.9 (Pin_9), J3.2 (Pin_2), J4.2 (Pin_2)
Changed lines of the file:
@@
 $EndDescr
 $Comp
-L Connector_Generic_MountingPin:Conn_01x09_MountingPin J?
-U 1 1 5EFB52FF
-P 4750 2850
-F 0 "J?" H 4838 2814 50  0000 L CNN
-F 1 "Conn_01x09_MountingPin" H 4838 2723 50  0000 L CNN
-F 2 "" H 4750 2850 50  0001 C CNN
-F 3 "~" H 4750 2850 50  0001 C CNN
-	1    4750 2850
+L Connector_Generic:Conn_01x09 J2
+U 1 1 5EFF586F
+P 3700 4250
+F 0 "J2" H 3780 4292 50  0000 L CNN
+F 1 "Digital pins" H 3780 4201 50  0000 L CNN
+F 2 "Connector_PinHeader_2.54mm:PinHeader_1x09_P2.54mm_Vertical" H 3700 4250 50  0001 C CNN
+F 3 "~" H 3700 4250 50  0001 C CNN
+	1    3700 4250
 	1    0    0    -1
 $EndComp
 $Comp
-L Connector_Generic_MountingPin:Conn_01x04_MountingPin J?
-U 1 1 5EFB5F86
-P 6300 2850
-F 0 "J?" H 6388 2764 50  0000 L CNN
-F 1 "Conn_01x04_MountingPin" H 6388 2673 50  0000 L CNN
-F 2 "" H 6300 2850 50  0001 C CNN
-F 3 "~" H 6300 2850 50  0001 C CNN
-	1    6300 2850
+L Connector_Generic:Conn_01x04 J1
+U 1 1 5EFF6E34
+P 3700 3050
+F 0 "J1" H 3780 3042 50  0000 L CNN
+F 1 "Serial" H 3780 2951 50  0000 L CNN
+F 2 "Connector_PinHeader_2.54mm:PinHeader_1x04_P2.54mm_Vertical" H 3700 3050 50  0001 C CNN
+F 3 "~" H 3700 3050 50  0001 C CNN
+	1    3700 3050
 	1    0    0    -1
 $EndComp
 $Comp
-L Connector_Generic:Conn_02x03_Odd_Even J?
-U 1 1 5EFB8292
-P 4700 4100
-F 0 "J?" H 4750 4417 50  0000 C CNN
-F 1 "Conn_02x03_Odd_Even" H 4750 4326 50  0000 C CNN
-F 2 "" H 4700 4100 50  0001 C CNN
-F 3 "~" H 4700 4100 50  0001 C CNN
-	1    4700 4100
+L Connector_Generic:Conn_01x04 J4
+U 1 1 5EFF7A80
+P 5300 3000
+F 0 "J4" H 5380 2992 50  0000 L CNN
+F 1 "I2C" H 5380 2901 50  0000 L CNN
+F 2 "Connector_PinHeader_2.54mm:PinHeader_1x04_P2.54mm_Vertical" H 5300 3000 50  0001 C CNN
+F 3 "~" H 5300 3000 50  0001 C CNN
+	1    5300 3000
 	1    0    0    -1
 $EndComp
 $Comp
-L Connector_Generic_MountingPin:Conn_01x04_MountingPin J?
-U 1 1 5EFB97C4
-P 6350 3850
-F 0 "J?" H 6438 3764 50  0000 L CNN
-F 1 "Conn_01x04_MountingPin" H 6438 3673 50  0000 L CNN
-F 2 "" H 6350 3850 50  0001 C CNN
-F 3 "~" H 6350 3850 50  0001 C CNN
-	1    6350 3850
+L Connector_Generic:Conn_02x03_Odd_Even J3
+U 1 1 5EFF865F
+P 5250 4150
+F 0 "J3" H 5300 4467 50  0000 C CNN
+F 1 "ICSP" H 5300 4376 50  0000 C CNN
+F 2 "Connector_PinHeader_2.54mm:PinHeader_2x03_P2.54mm_Vertical" H 5250 4150 50  0001 C CNN
+F 3 "~" H 5250 4150 50  0001 C CNN
+	1    5250 4150
 	1    0    0    -1
 $EndComp
+Text HLabel 5050 4050 0    50   Output ~ 0
+MISO
+Text HLabel 5050 4150 0    50   BiDi ~ 0
+SCK
+Text HLabel 5050 4250 0    50   Output ~ 0
+RST
+Text HLabel 5550 4050 2    50   Input ~ 0
+VCC
+Text HLabel 5550 4150 2    50   Input ~ 0
+MOSI
+Text HLabel 5550 4250 2    50   Input ~ 0
+GND
+Text HLabel 5100 2900 0    50   Input ~ 0
+GND
+Text HLabel 5100 3000 0    50   Input ~ 0
+VCC
+Text HLabel 5100 3100 0    50   BiDi ~ 0
+SDA
+Text HLabel 5100 3200 0    50   BiDi ~ 0
+SCK
+Text HLabel 3500 2950 0    50   Input ~ 0
+GND
+Text HLabel 3500 3050 0    50   Input ~ 0
+VCC
+Text HLabel 3500 3150 0    50   Input ~ 0
+RX
+Text HLabel 3500 3250 0    50   Output ~ 0
+TX
+Text HLabel 3500 3850 0    50   BiDi ~ 0
+D2
+Text HLabel 3500 3950 0    50   BiDi ~ 0
+D3
+Text HLabel 3500 4050 0    50   BiDi ~ 0
+D4
+Text HLabel 3500 4150 0    50   BiDi ~ 0
+D5
+Text HLabel 3500 4250 0    50   BiDi ~ 0
+D6
+Text HLabel 3500 4350 0    50   BiDi ~ 0
+D7
+Text HLabel 3500 4450 0    50   BiDi ~ 0
+D8
+Text HLabel 3500 4550 0    50   Input ~ 0
+GND
+Text HLabel 3500 4650 0    50   Input ~ 0
+VCC
 $EndSCHEMATC

Commit message: comments and netlist
Other:
- note added: "GPIO Connector"
- note added: "I2C - Connector\n"
- note added: "SPI connector\n"
- note added: "Serial connector\n"
- moved on the sheet: J3, J4
Changed lines of the file:
@@
 L Connector_Generic:Conn_01x04 J4
 U 1 1 5EFF7A80
-P 5300 3000
-F 0 "J4" H 5380 2992 50  0000 L CNN
-F 1 "I2C" H 5380 2901 50  0000 L CNN
-F 2 "Connector_PinHeader_2.54mm:PinHeader_1x04_P2.54mm_Vertical" H 5300 3000 50  0001 C CNN
-F 3 "~" H 5300 3000 50  0001 C CNN
-	1    5300 3000
+P 5300 3100
+F 0 "J4" H 5380 3092 50  0000 L CNN
+F 1 "I2C" H 5380 3001 50  0000 L CNN
+F 2 "Connector_PinHeader_2.54mm:PinHeader_1x04_P2.54mm_Vertical" H 5300 3100 50  0001 C CNN
+F 3 "~" H 5300 3100 50  0001 C CNN
+	1    5300 3100
 	1    0    0    -1
 $EndComp
@@
 L Connector_Generic:Conn_02x03_Odd_Even J3
 U 1 1 5EFF865F
-P 5250 4150
-F 0 "J3" H 5300 4467 50  0000 C CNN
-F 1 "ICSP" H 5300 4376 50  0000 C CNN
-F 2 "Connector_PinHeader_2.54mm:PinHeader_2x03_P2.54mm_Vertical" H 5250 4150 50  0001 C CNN
-F 3 "~" H 5250 4150 50  0001 C CNN
-	1    5250 4150
+P 5200 4300
+F 0 "J3" H 5250 4617 50  0000 C CNN
+F 1 "ICSP" H 5250 4526 50  0000 C CNN
+F 2 "Connector_PinHeader_2.54mm:PinHeader_2x03_P2.54mm_Vertical" H 5200 4300 50  0001 C CNN
+F 3 "~" H 5200 4300 50  0001 C CNN
+	1    5200 4300
 	1    0    0    -1
 $EndComp
-Text HLabel 5050 4050 0    50   Output ~ 0
+Text HLabel 5000 4200 0    50   Output ~ 0
 MISO
-Text HLabel 5050 4150 0    50   BiDi ~ 0
+Text HLabel 5000 4300 0    50   BiDi ~ 0
 SCK
-Text HLabel 5050 4250 0    50   Output ~ 0
+Text HLabel 5000 4400 0    50   Output ~ 0
 RST
-Text HLabel 5550 4050 2    50   Input ~ 0
+Text HLabel 5500 4200 2    50   Input ~ 0
 VCC
-Text HLabel 5550 4150 2    50   Input ~ 0
+Text HLabel 5500 4300 2    50   Input ~ 0
 MOSI
-Text HLabel 5550 4250 2    50   Input ~ 0
-GND
-Text HLabel 5100 2900 0    50   Input ~ 0
+Text HLabel 5500 4400 2    50   Input ~ 0
 GND
 Text HLabel 5100 3000 0    50   Input ~ 0
+GND
+Text HLabel 5100 3100 0    50   Input ~ 0
 VCC
-Text HLabel 5100 3100 0    50   BiDi ~ 0
+Text HLabel 5100 3200 0    50   BiDi ~ 0
 SDA
-Text HLabel 5100 3200 0    50   BiDi ~ 0
+Text HLabel 5100 3300 0    50   BiDi ~ 0
 SCK
 Text HLabel 3500 2950 0    50   Input ~ 0
@@
 Text HLabel 3500 4650 0    50   Input ~ 0
 VCC
+Wire Notes Line
+	3100 2550 3100 4950
+Wire Notes Line
+	3100 4950 5800 4950
+Wire Notes Line
+	5800 4950 5800 2550
+Wire Notes Line
+	5800 2550 3100 2550
+Text Notes 3350 2800 0    50   ~ 0
+Serial connector\n
+Text Notes 4900 2800 0    50   ~ 0
+I2C - Connector\n
+Text Notes 3400 3700 0    50   ~ 0
+GPIO Connector
+Text Notes 5000 3850 0    50   ~ 0
+SPI connector\n
 $EndSCHEMATC
