File: BACEE.kicad_pcb_2_layer.kicad_pcb (KiCad board)
At the start: 2 copper layers, 42.7 x 29 mm, 17 parts, among them J1 Serial, J2 Digital pins, J3 ICSP, J4 I2C, U1 24LC1025, U2 24LC1025, U3 DS1337_KTH, U4 ATMEGA328P-AU, Y1 Crystal 32MHz, Y2 Crystal 16MHz

Commit message: fully routed in 2 layers - saved a copy
Routing:
- net GND: track 0.00 -> 155.5 mm, vias 0 -> 1
- net VCC: track 0.00 -> 133.2 mm, vias 0 -> 2
- net SCK: track 0.00 -> 102.5 mm
- net SDA: track 0.00 -> 64.5 mm, vias 0 -> 1
- net Net-(C1-Pad1): track 0.00 -> 48.7 mm
- net RST: track 0.00 -> 46.3 mm, vias 0 -> 1
- net MISO: track 0.00 -> 33.8 mm, vias 0 -> 1
- net TX: track 0.00 -> 33.3 mm, vias 0 -> 1
- net RX: track 0.00 -> 30.0 mm, vias 0 -> 1
- net Net-(D1-Pad2): track 0.00 -> 23.7 mm
- net Net-(C2-Pad1): track 0.00 -> 23.7 mm, vias 0 -> 2
- net ADDS2: track 0.00 -> 23.6 mm
- net Net-(U3-Pad1): track 0.00 -> 21.8 mm
- net D2: track 0.00 -> 20.9 mm
- net MOSI: track 0.00 -> 16.8 mm, vias 0 -> 1
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